Commit message: Add model

File: urdf/basic_International_ROV.urdf (robot description, URDF)
Before this commit: robot myCameraStereo, 5 links, 4 joints
Links:
- link cameras: geometry collision box size=0.05 0.05 0.05; visual mesh filename=file://$(find project_aur_controller)/meshes/Model_ROV.stl scale=0.5 0.5 0.5
